Commit message: rviz editing...

File: robot_description/urdf/my_robot.urdf (robot description, URDF)
Before this commit: robot my_robot, 3 links, 2 joints
Links:
- added link wheel_4, mass 10; collision cylinder length=0.05 radius=0.05; visual cylinder length=0.05 radius=0.05
- added link wheel_free, mass 5; collision cylinder length=0.025 radius=0.031; visual cylinder length=0.025 radius=0.031
- link base_link: mass None -> 50; geometry collision box size=0.175 .11 0.05; visual box size=0.175 0.11 0.05
- link wheel_left: mass None -> 5; geometry collision cylinder length=0.05 radius=0.05; visual cylinder length=0.025 radius=0.031
- link wheel_right: mass None -> 5; geometry collision cylinder length=0.025 radius=0.031; visual cylinder length=0.025 radius=0.031
Joints:
- removed joint base_to_wheel_left
- removed joint base_to_wheel_right
- added joint base_to_wheel1: type fixed, parent base_link, child wheel_right, origin xyz=0 0 0
- added joint base_to_wheel2: type fixed, parent base_link, child wheel_left, origin xyz=0 0 0
- added joint base_to_wheel3: type fixed, parent base_link, child wheel_free, origin xyz=0 0 0
- added joint base_to_wheel4: type fixed, parent base_link, child wheel_4, origin xyz=0 0 0

Commit message: ...

File: robot_description/urdf/my_robot.urdf (robot description, URDF)
Before this commit: robot my_robot, 5 links, 4 joints
Links:
- removed link wheel_4
- link base_link: geometry collision box size=0.11 .175 0.05; visual box size=0.11 0.175 0.05
- link wheel_free: geometry collision cylinder length=0.01 radius=0.015; visual cylinder length=0.025 radius=0.031
Joints:
- removed joint base_to_wheel1
- removed joint base_to_wheel2
- removed joint base_to_wheel3
- removed joint base_to_wheel4
- added joint base_to_wheel_free: type fixed, parent base_link, child wheel_free, origin xyz=0 0.055 0
- added joint base_to_wheel_left: type fixed, parent base_link, child wheel_left, origin xyz=-0.04375 -0.04375 0
- added joint base_to_wheel_right: type fixed, parent base_link, child wheel_right, origin xyz=0.04375 -0.04375 0
