Commit message: Rename and order packages

File: my_robot_description/robots/my_robot_circles_kinect.urdf.xacro (robot description, xacro)
@@ -6,6 +6,5 @@
 -->
 <robot name="turtlebot" xmlns:xacro="http://ros.org/wiki/xacro">
-<!--  <xacro:include filename="$(find turtlebot_description)/urdf/turtlebot_library.urdf.xacro" /> -->
-  <xacro:include filename="$(find chefbot_description)/urdf/chefbot_rviz_library.urdf.xacro" />
+  <xacro:include filename="$(find my_robot_description)/urdf/my_robot_library.urdf.xacro" />
   <kobuki/>
   <stack_hexagons parent="base_link"/>

File: my_robot_description/urdf/my_robot_base.urdf.xacro (robot description, xacro)
@@ -6,8 +6,8 @@
       kobuki_description/launch/view_model.launch
  -->
-<robot name="kobuki" xmlns:xacro="http://ros.org/wiki/xacro">
-  <xacro:include filename="$(find chefbot_description)/urdf/common_properties.urdf.xacro"/>
-  <xacro:include filename="$(find chefbot_description)/urdf/chefbot_base_gazebo.urdf.xacro"/>
-  <!-- Kobuki -->
+<robot name="my_robot" xmlns:xacro="http://ros.org/wiki/xacro">
+  <xacro:include filename="$(find my_robot_description)/urdf/common_properties.urdf.xacro"/>
+  <xacro:include filename="$(find my_robot_description)/urdf/my_robot_base_gazebo.urdf.xacro"/>
+  <!-- my_robot -->
   <xacro:macro name="kobuki">
     <link name="base_footprint"/>
@@ -30,5 +30,5 @@
         <geometry>
           <!-- new mesh -->
-          <mesh filename="package://chefbot_description/meshes/base_plate.dae" />
+          <mesh filename="package://my_robot_description/meshes/base_plate.dae" />
         </geometry>
 <!--        <origin xyz="0.001 0 0.05199" rpy="0 0 ${M_PI/2}"/> -->
@@ -59,12 +59,12 @@
     <joint name="wheel_left_joint" type="continuous">
       <parent link="base_link"/>
-      <child link="wheel_left_link"/>
+      <child link="my_robot_wheel_left_link"/>
       <origin xyz="0 ${0.28/2} 0.026" rpy="${-M_PI/2} 0 0"/>
       <axis xyz="0 0 1"/>
     </joint>
-    <link name="wheel_left_link">
+    <link name="my_robot_wheel_left_link">
       <visual>
         <geometry>
-          <mesh filename="package://chefbot_description/meshes/wheel.dae"/>
+          <mesh filename="package://my_robot_description/meshes/wheel.dae"/>
         </geometry>
         <origin xyz="0 0 0" rpy="0 0 0"/>
@@ -86,12 +86,12 @@
     <joint name="wheel_right_joint" type="continuous">
       <parent link="base_link"/>
-      <child link="wheel_right_link"/>
+      <child link="my_robot_wheel_right_link"/>
       <origin xyz="0.00 -${0.28/2} 0.026" rpy="${-M_PI/2} 0 0"/>
       <axis xyz="0 0 1"/>
     </joint>
-    <link name="wheel_right_link">
+    <link name="my_robot_wheel_right_link">
       <visual>
         <geometry>
-          <mesh filename="package://chefbot_description/meshes/wheel.dae"/>
+          <mesh filename="package://my_robot_description/meshes/wheel.dae"/>
         </geometry>
         <origin xyz="0 0 0" rpy="0 0 0"/>
@@ -111,10 +111,124 @@
       </inertial>
     </link>
+<!--
+	  <link name="left_axle_link">
+	    <inertial>
+	      <origin xyz="0 0 0"/>
+	      <mass value="0.01" />
+	      <inertia ixx="0.001" ixy="0.0" ixz="0.0"
+	        iyy="0.001" iyz="0.0" izz="0.001" />
+	    </inertial>
+	    <visual>
+	      <origin xyz="0 0 0" rpy="0 1.5707 1.5707" />
+	      <geometry>
+            <cylinder radius="0.00635" length = "0.00635"/>
+	      </geometry>
+          <material name ="light_grey" />
+	    </visual>
+	    <collision>
+	      <origin xyz="0 0 0" rpy="0 1.5707 1.5707" />
+	      <geometry>
+            <cylinder radius="0.00635" length = "0.00635"/>
+	      </geometry>
+	    </collision>
+	  </link>
+	  <joint name="left_axle_joint" type="fixed">
+	    <origin xyz="0 0.171475 0.0178" rpy="0 0 0"/>
+	    <parent link="base_link"/>
+	    <child link="left_axle_link"/>
+	    <axis xyz="0 1 0"/>
+	  </joint>
+	  <link name="right_axle_link">
+	    <inertial>
+	      <origin xyz="0 0 0"/>
+	      <mass value="0.01" />
+	      <inertia ixx="0.001" ixy="0.0" ixz="0.0"
+	        iyy="0.001" iyz="0.0" izz="0.001" />
+	    </inertial>
+	    <visual>
+	      <origin xyz="0 0 0" rpy="0 1.5707 1.5707" />
+	      <geometry>
+            <cylinder radius="0.00635" length = "0.00635"/>
+	      </geometry>
+          <material name ="light_grey" />
+	    </visual>
+	    <collision>
+	      <origin xyz="0 0 0" rpy="0 1.5707 1.5707" />
+	      <geometry>
+            <cylinder radius="0.00635" length = "0.00635"/>
+	      </geometry>
+	    </collision>
+	  </link>
+	  <joint name="right_axle_joint" type="fixed">
+	    <origin xyz="0 -0.171475 0.0178" rpy="0 0 0"/>
+	    <parent link="base_link"/>
+	    <child link="right_axle_link"/>
+	    <axis xyz="0 1 0"/>
+	  </joint>
+	  <link name="left_wheel_link">
+	    <inertial>
+	      <origin xyz="0 0 0"/>
+	      <mass value="0.01" />
+	      <inertia ixx="0.001" ixy="0.0" ixz="0.0"
+	        iyy="0.001" iyz="0.0" izz="0.001" />
+	    </inertial>
+	    <visual>
+	      <origin xyz="0 0 0" rpy="0 1.5707 1.5707" />
+	      <geometry>
+            <cylinder radius="0.0762" length = "0.03175"/>
+	      </geometry>
+          <material name ="black" />
+	    </visual>
+	    <collision>
+	      <origin xyz="0 0 0" rpy="0 1.5707 1.5707" />
+	      <geometry>
+            <cylinder radius="0.0762" length = "0.03175"/>
+	      </geometry>
+	    </collision>
+	  </link>
+        -->
+<!--	  <joint name="left_wheel_joint" type="fixed">
+	    <origin xyz="0 0.01905 0" rpy="0 0 0"/>
+	    <parent link="left_axle_link"/>
+	    <child link="left_wheel_link"/>
+	    <axis xyz="0 1 0"/>
+	  </joint>
+	  <link name="right_wheel_link">
+	    <inertial>
+	      <origin xyz="0 0 0"/>
+	      <mass value="0.01" />
+	      <inertia ixx="0.001" ixy="0.0" ixz="0.0"
+	        iyy="0.001" iyz="0.0" izz="0.001" />
+	    </inertial>
+	    <visual>
+	      <origin xyz="0 0 0" rpy="0 1.5707 1.5707" />
+	      <geometry>
+            <cylinder radius="0.0762" length = "0.03175"/>
+	      </geometry>
+          <material name ="black" />
+	    </visual>
+	    <collision>
+	      <origin xyz="0 0 0" rpy="0 1.5707 1.5707" />
+	      <geometry>
+            <cylinder radius="0.0762" length = "0.03175"/>
+	      </geometry>
+	    </collision>
+	  </link>
+	-->
+        <!-- Fixed because we never rotate it anyway, it is just for show -->
+        <!-- NOTE This may prevent gazebo from working with this model -->
+<!--	  <joint name="right_wheel_joint" type="fixed">
+	    <origin xyz="0 -0.01905 0" rpy="0 0 0"/>
+	    <parent link="right_axle_link"/>
+	    <child link="right_wheel_link"/>
+	    <axis xyz="0 1 0"/>
+	  </joint>
+-->
     <joint name="caster_front_joint" type="fixed">
       <parent link="base_link"/>
-      <child link="caster_front_link"/>
+      <child link="my_robot_caster_front_link"/>
       <origin xyz="0.115 0.0 0.007" rpy="${-M_PI/2} 0 0"/>
     </joint>
-    <link name="caster_front_link">
+    <link name="my_robot_caster_front_link">
       <collision>
         <geometry>
@@ -131,10 +245,10 @@
       </inertial>
     </link>
-    <joint name="caster_back_joint" type="fixed">
-      <parent link="base_link"/>
-      <child link="caster_back_link"/>
+    <joint name="my_robot_caster_back_joint" type="fixed">
+      <parent link="base_link"/>
+      <child link="my_robot_caster_back_link"/>
       <origin xyz="-0.135 0.0 0.009" rpy="${-M_PI/2} 0 0"/>
     </joint>
-    <link name="caster_back_link">
+    <link name="my_robot_caster_back_link">
       <collision>
         <geometry>

File: my_robot_description/urdf/sensors/asus_xtion_pro.urdf.xacro (robot description, xacro)
@@ -2,5 +2,5 @@
 <robot name="sensor_asus_xtion_pro" xmlns:xacro="http://ros.org/wiki/xacro">
   <xacro:include filename="$(find turtlebot_description)/urdf/turtlebot_gazebo.urdf.xacro"/>
-  <xacro:include filename="$(find turtlebot_description)/urdf/turtlebot_properties.urdf.xacro"/>f.xacro"/>
+  <xacro:include filename="$(find turtlebot_description)/urdf/turtlebot_properties.urdf.xacro"/>
   <!-- Xacro properties -->
   <xacro:property name="M_SCALE" value="0.001"/>

File: my_robot_description/urdf/sensors/kinect.urdf.xacro (robot description, xacro)
@@ -1,6 +1,6 @@
 <?xml version="1.0"?>
 <robot name="sensor_kinect" xmlns:xacro="http://ros.org/wiki/xacro">
-  <xacro:include filename="$(find chefbot_description)/urdf/chefbot_gazebo.urdf.xacro"/>
-  <xacro:include filename="$(find chefbot_description)/urdf/chefbot_properties.urdf.xacro"/>
+  <xacro:include filename="$(find my_robot_description)/urdf/my_robot_gazebo.urdf.xacro"/>
+  <xacro:include filename="$(find my_robot_description)/urdf/my_robot_properties.urdf.xacro"/>
   <!-- Parameterised in part by the values in turtlebot_properties.urdf.xacro -->
   <xacro:macro name="sensor_kinect" params="parent">
