Commit message: Add Velodyne model - needs modifications

File: my_robot_description/urdf/inertias.xacro (robot description, xacro)
@@ -5,5 +5,6 @@
 <robot xmlns:xacro="http://www.ros.org/wiki/xacro">
   <xacro:macro name="cylinder_inertia" params="m r h">
-    <inertia  ixx="${m*(3*r*r+h*h)/12}"
+    <inertia
+          ixx="${m*(3*r*r+h*h)/12}"
     			ixy = "0"
     			ixz = "0"
@@ -14,5 +15,6 @@
   </xacro:macro>
   <xacro:macro name="box_inertia" params="m x y z">
-    <inertia  ixx="${m*(y*y+z*z)/12}"
+    <inertia
+          ixx="${m*(y*y+z*z)/12}"
     			ixy = "0"
     			ixz = "0"
@@ -23,5 +25,6 @@
   </xacro:macro>
   <xacro:macro name="sphere_inertia" params="m r">
-    <inertia  ixx="${2*m*r*r/5}"
+    <inertia
+          ixx="${2*m*r*r/5}"
     			ixy = "0"
     			ixz = "0"

File: my_robot_description/urdf/my_robot.xacro (robot description, xacro)
@@ -12,6 +12,8 @@
 	<!-- Import Rviz colors -->
 	<xacro:include filename="$(find my_robot_description)/urdf/materials.xacro" />
+	<!-- Gazebo aspects of the robot -->
 	<xacro:include filename="$(find my_robot_description)/urdf/my_robot.gazebo" />
-	<xacro:include filename="$(find my_robot_description)/urdf/macros.xacro" />
+	<!-- Inertia matrices -->
+	<xacro:include filename="$(find my_robot_description)/urdf/inertias.xacro" />
 	<!-- Used for fixing robot to Gazebo 'chassis' -->
 	<link name="base_footprint" />
@@ -25,7 +27,4 @@
 					rpy="0 0 0"/>
 			<geometry>
-				<!--box size="${chassisLength}
-						   ${chassisWidth}
-						   ${chassisHeight}"/-->
 				<mesh filename="package://my_robot_description/meshes/chassis.dae" />
 			</geometry>
@@ -59,5 +58,4 @@
 					rpy="0 0 0"/>
 			<geometry>
-				<!--sphere radius="${casterRadius}"/-->
 				<mesh filename="package://my_robot_description/meshes/caster_wheel.dae" />
 	  		</geometry>
@@ -67,5 +65,4 @@
 					rpy="0 0 0"/>
 			<geometry>
-				<!--sphere radius="${casterRadius}"/-->
 				<mesh filename="package://my_robot_description/meshes/caster_wheel.dae" />
 			</geometry>
@@ -83,35 +80,7 @@
 	<wheel lr="left" tY="-1"/>
 	<wheel lr="right" tY="1"/>
-	<!--joint name="camera_joint" type="fixed">
-		<origin xyz="${-cameraSize+chassisLength/2} 0 ${cameraSize+wheelRadius+cameraSize/2}" rpy="0 0 0"/>
-		<parent link="chassis"/>
-		<child link="camera"/>
-	</joint>
-	<link name="camera">
-		<collision>
-			<origin xyz="0 0 0" rpy="0 0 0"/>
-			<geometry>
-				<box size="${cameraSize}
-						   ${cameraSize}
-						   ${cameraSize}"/>
-			</geometry>
-		</collision>
-		<visual>
-			<origin xyz="0 0 0" rpy="0 0 0"/>
-			<geometry>
-				<box size="${cameraSize}
-						   ${cameraSize}
-						   ${cameraSize}"/>
-			</geometry>
-			<material name="blue"/>
-		</visual>
-		<inertial>
-			<mass value="${cameraMass}" />
-			<origin xyz="0 0 0" rpy="0 0 0"/>
-			<box_inertia m="${cameraMass}"
-						 x="${cameraSize}"
-						 y="${cameraSize}"
-						 z="${cameraSize}" />
-		</inertial>
-	</link-->
+	<!-- Including Velodyne model -->
+	<xacro:include filename="$(find my_robot_description)/urdf/velodyne.xacro" />
+	<!-- Camera model -->
+	<!--xacro:include filename="$(find my_robot_description)/urdf/camera.xacro" /-->
 </robot>

File: my_robot_description/urdf/my_robot_properties.xacro (robot description, xacro)
@@ -1,17 +1,28 @@
 <?xml version="1.0"?>
 <robot xmlns:xacro="http://www.ros.org/wiki/xacro">
+	<!-- Constants -->
 	<xacro:property name="PI" value="3.1415926535897931"/>
+	<!-- Chassis properties -->
 	<xacro:property name="chassisHeight" value="0.0623"/>
 	<xacro:property name="chassisLength" value="0.198"/>
 	<xacro:property name="chassisWidth" value="0.119"/>
 	<xacro:property name="chassisMass" value="0.15"/>
+	<!-- Caster wheel properties -->
 	<xacro:property name="casterRadius" value="0.021"/>
 	<xacro:property name="casterMass" value="0.09"/>
 	<xacro:property name="casterOffsetX" value="0.091"/>
+	<!-- Differential-drive wheels properties -->
 	<xacro:property name="wheelWidth" value="0.026"/>
 	<xacro:property name="wheelRadius" value="0.032"/>
 	<xacro:property name="wheelMass" value="0.05"/>
 	<xacro:property name="wheelOffsetY" value="0.047"/>
-	<!--xacro:property name="cameraSize" value="0.05"/>
-	<xacro:property name="cameraMass" value="0.1"/-->
+	<!-- Velodyne properties -->
+	<xacro:property name="velodyneLengthBottom" value="0.05867"/>
+	<xacro:property name="velodyneLengthTop" value="0.07357"/>
+	<xacro:property name="velodyneMassBottom" value="1.2"/>
+	<xacro:property name="velodyneMassTop" value="0.1"/>
+	<xacro:property name="velodyneRadius" value="0.04267"/>
+	<!-- Camera properties -->
+	<xacro:property name="cameraSize" value="0.05"/>
+	<xacro:property name="cameraMass" value="0.1"/>
 </robot>
