Commit message: Almost working gazebo & rviz simulations

File: my_robot_description/urdf/macros.xacro (robot description, xacro)
@@ -77,10 +77,16 @@
       <joint_properties damping="0.0" friction="0.0"/>
     </joint>
+<!--
+  http://gazebosim.org/tutorials/?tut=ros_control
+-->
     <transmission name="${lr}_trans">
       <type>transmission_interface/SimpleTransmission</type>
-      <joint name="${lr}_wheel_hinge"/>
+      <joint name="${lr}_wheel_hinge">
+        <hardwareInterface>hardware_interface/EffortJointInterface</hardwareInterface>
+      </joint>
       <actuator name="${lr}Motor">
-        <hardwareInterface>EffortJointInterface</hardwareInterface>
+        <hardwareInterface>hardware_interface/EffortJointInterface</hardwareInterface>
         <mechanicalReduction>10</mechanicalReduction>
+        <!--mechanicalReduction>1</mechanicalReduction-->
       </actuator>
     </transmission>

File: my_robot_description/urdf/materials.xacro (robot description, xacro)
@@ -1,5 +1,5 @@
 <?xml version="1.0"?>
 <!--
-	definition of the materials used (mostly colors)
+	definition of the materials used
 -->
 <robot>

File: my_robot_description/urdf/my_robot.xacro (robot description, xacro)
@@ -2,15 +2,7 @@
 <!--
 	http://www.generationrobots.com/blog/en/2015/02/robotic-simulation-scenarios-with-gazebo-and-ros/#create your own robot model
-	http://gazebosim.org/tutorials?cat=guided_b&tut=guided_b3
-	https://github.com/HumaRobotics/mybot_gazebo_tutorial
-	https://github.com/jaypatravali/mybot_gazebo
-	#######################################################
-	To check whether the sintax is fine or whether it have errors:
-    $ check_urdf my_robot.urdf
-    To get the Graphviz in pdf:
-    $ urdf_to_graphviz my_robot.urdf
 	#######################################################
     To run:
-    $ roslaunch my_robot_gazebo simple.launch
+    $ roslaunch my_robot_gazebo my_robot_world.launch
     $ rosrun turtlebot_teleop turtlebot_teleop_key /turtlebot_teleop/cmd_vel:=/my_robot/cmd_vel
 -->
@@ -24,5 +16,6 @@
 	<xacro:property name="casterMass" value="0.1"/>
 	<xacro:property name="wheelWidth" value="0.026"/>
-	<xacro:property name="wheelRadius" value="0.037"/>
+	<xacro:property name="wheelRadius" value="0.05"/>
+	<!--xacro:property name="wheelRadius" value="0.037"/-->
 	<xacro:property name="wheelPos" value="0.11"/>
 	<xacro:property name="wheelMass" value="0.01"/>
@@ -30,9 +23,11 @@
 	<xacro:property name="cameraMass" value="0.1"/-->
 	<xacro:include filename="$(find my_robot_description)/urdf/my_robot.gazebo" />
+	<!-- Import Rviz colors -->
 	<xacro:include filename="$(find my_robot_description)/urdf/materials.xacro" />
 	<xacro:include filename="$(find my_robot_description)/urdf/macros.xacro" />
-	<link name="footprint" />
+	<!-- Used for fixing robot to Gazebo 'chassis' -->
+	<link name="world" />
 	<joint name="base_joint" type="fixed">
-		<parent link="footprint"/>
+		<parent link="world"/>
 		<child link="chassis"/>
 	</joint>

Commit message: Big progress, need to adjust to real robot

File: my_robot_description/urdf/macros.xacro (robot description, xacro)
@@ -44,7 +44,8 @@
         <origin xyz="0 0 0" rpy="0 ${PI/2} ${PI/2}" />
         <geometry>
-          <cylinder
+          <!--cylinder
             length="${wheelWidth}"
-            radius="${wheelRadius}"/>
+            radius="${wheelRadius}"/-->
+          <mesh filename="package://my_robot_description/meshes/${lr}_wheel.dae" />
         </geometry>
         <material name="black"/>

File: my_robot_description/urdf/my_robot.xacro (robot description, xacro)
@@ -9,5 +9,17 @@
 <robot name="my_robot" xmlns:xacro="http://www.ros.org/wiki/xacro">
 	<xacro:property name="PI" value="3.1415926535897931"/>
-	<xacro:property name="chassisHeight" value="0.08"/>
+	<xacro:property name="chassisHeight" value="0.1"/>
+	<xacro:property name="chassisLength" value="0.4"/>
+	<xacro:property name="chassisWidth" value="0.2"/>
+	<xacro:property name="chassisMass" value="50"/>
+	<xacro:property name="casterRadius" value="0.05"/>
+	<xacro:property name="casterMass" value="5"/>
+	<xacro:property name="wheelWidth" value="0.05"/>
+	<xacro:property name="wheelRadius" value="0.1"/>
+	<xacro:property name="wheelPos" value="0.2"/>
+	<xacro:property name="wheelMass" value="5"/>
+	<xacro:property name="cameraSize" value="0.05"/>
+	<xacro:property name="cameraMass" value="0.1"/>
+	<!--xacro:property name="chassisHeight" value="0.08"/>
 	<xacro:property name="chassisLength" value="0.175"/>
 	<xacro:property name="chassisWidth" value="0.11"/>
@@ -16,9 +28,8 @@
 	<xacro:property name="casterMass" value="0.1"/>
 	<xacro:property name="wheelWidth" value="0.026"/>
-	<xacro:property name="wheelRadius" value="0.05"/>
-	<!--xacro:property name="wheelRadius" value="0.037"/-->
+	<xacro:property name="wheelRadius" value="0.037"/>
 	<xacro:property name="wheelPos" value="0.11"/>
 	<xacro:property name="wheelMass" value="0.01"/>
-	<!--xacro:property name="cameraSize" value="0.05"/>
+	<xacro:property name="cameraSize" value="0.05"/>
 	<xacro:property name="cameraMass" value="0.1"/-->
 	<xacro:include filename="$(find my_robot_description)/urdf/my_robot.gazebo" />
@@ -42,10 +53,6 @@
 			<origin xyz="0 0 ${wheelRadius}" rpy="0 0 0"/>
 			<geometry>
-				<box size="${chassisLength} ${chassisWidth} ${chassisHeight}"/>
-				<!--mesh>
-					<uri>
-						file://../meshes/chassis_resized.dae
-					</uri>
-				</mesh-->
+				<!--box size="${chassisLength} ${chassisWidth} ${chassisHeight}"/-->
+				<mesh filename="package://my_robot_description/meshes/chassis.dae" />
 			</geometry>
 			<material name="orange"/>
@@ -68,10 +75,10 @@
 	  		</geometry>
 		</collision>
-		<visual>
+		<!--visual>
 			<origin xyz="${casterRadius-chassisLength/2} 0 ${casterRadius-chassisHeight+wheelRadius}" rpy="0 0 0"/>
 			<geometry>
 				<sphere radius="${casterRadius}"/>
 			</geometry>
-		</visual>
+		</visual-->
 		<inertial>
 			<origin xyz="${casterRadius-chassisLength/2} 0 ${casterRadius-chassisHeight+wheelRadius}" rpy="0 0 0"/>

Commit message: Solved jittering, but still incorrect Gazebo model

File: my_robot_description/urdf/macros.xacro (robot description, xacro)
@@ -72,8 +72,11 @@
       <child link="${lr}_wheel"/>
       <origin
-        xyz="${+wheelPos-chassisLength/4} ${tY*wheelWidth/2+tY*chassisWidth/2} ${wheelRadius}"
-        rpy="0 0 0" />
+        xyz = "${+wheelPos-chassisLength/4}
+               ${tY*wheelWidth/2+tY*chassisWidth/2}
+               ${wheelRadius}"
+        rpy = "0 0 0" />
       <axis xyz="0 1 0" rpy="0 0 0" />
-      <limit effort="100" velocity="100"/>
+      <!--limit effort="100" velocity="100"/-->
+      <limit effort="10" velocity="10"/>
       <joint_properties damping="0.0" friction="0.0"/>
     </joint>
@@ -88,6 +91,6 @@
       <actuator name="${lr}Motor">
         <hardwareInterface>hardware_interface/EffortJointInterface</hardwareInterface>
-        <mechanicalReduction>10</mechanicalReduction>
-        <!--mechanicalReduction>1</mechanicalReduction-->
+        <!--mechanicalReduction>10</mechanicalReduction-->
+        <mechanicalReduction>1</mechanicalReduction>
       </actuator>
     </transmission>

File: my_robot_description/urdf/my_robot.xacro (robot description, xacro)
@@ -9,28 +9,16 @@
 <robot name="my_robot" xmlns:xacro="http://www.ros.org/wiki/xacro">
 	<xacro:property name="PI" value="3.1415926535897931"/>
-	<xacro:property name="chassisHeight" value="0.1"/>
-	<xacro:property name="chassisLength" value="0.4"/>
-	<xacro:property name="chassisWidth" value="0.2"/>
-	<xacro:property name="chassisMass" value="50"/>
-	<xacro:property name="casterRadius" value="0.05"/>
-	<xacro:property name="casterMass" value="5"/>
-	<xacro:property name="wheelWidth" value="0.05"/>
-	<xacro:property name="wheelRadius" value="0.1"/>
-	<xacro:property name="wheelPos" value="0.2"/>
-	<xacro:property name="wheelMass" value="5"/>
+	<xacro:property name="chassisHeight" value="0.037"/>
+	<xacro:property name="chassisLength" value="0.175"/>
+	<xacro:property name="chassisWidth" value="0.142"/>
+	<xacro:property name="chassisMass" value="0.25"/>
+	<xacro:property name="casterRadius" value="0.0125"/>
+	<xacro:property name="casterMass" value="0.05"/>
+	<xacro:property name="wheelWidth" value="0.025"/>
+	<xacro:property name="wheelRadius" value="0.037"/>
+	<xacro:property name="wheelPos" value="0.036"/>
+	<xacro:property name="wheelMass" value="0.05"/>
 	<xacro:property name="cameraSize" value="0.05"/>
 	<xacro:property name="cameraMass" value="0.1"/>
-	<!--xacro:property name="chassisHeight" value="0.08"/>
-	<xacro:property name="chassisLength" value="0.175"/>
-	<xacro:property name="chassisWidth" value="0.11"/>
-	<xacro:property name="chassisMass" value="0.5"/>
-	<xacro:property name="casterRadius" value="0.025"/>
-	<xacro:property name="casterMass" value="0.1"/>
-	<xacro:property name="wheelWidth" value="0.026"/>
-	<xacro:property name="wheelRadius" value="0.037"/>
-	<xacro:property name="wheelPos" value="0.11"/>
-	<xacro:property name="wheelMass" value="0.01"/>
-	<xacro:property name="cameraSize" value="0.05"/>
-	<xacro:property name="cameraMass" value="0.1"/-->
 	<xacro:include filename="$(find my_robot_description)/urdf/my_robot.gazebo" />
 	<!-- Import Rviz colors -->
@@ -47,5 +35,7 @@
 			<origin xyz="0 0 ${wheelRadius}" rpy="0 0 0"/>
 			<geometry>
-				<box size="${chassisLength} ${chassisWidth} ${chassisHeight}"/>
+				<box size="${chassisLength}
+						   ${chassisWidth}
+						   ${chassisHeight}"/>
 			</geometry>
 		</collision>
@@ -56,10 +46,14 @@
 				<mesh filename="package://my_robot_description/meshes/chassis.dae" />
 			</geometry>
-			<material name="orange"/>
+			<material name="red"/>
 		</visual>
 		<inertial>
 			<origin xyz="0 0 ${wheelRadius}" rpy="0 0 0"/>
 			<mass value="${chassisMass}"/>
-			<box_inertia m="${chassisMass}" x="${chassisLength}" y="${chassisWidth}" z="${chassisHeight}"/>
+			<box_inertia
+				m="${chassisMass}"
+				x="${chassisLength}"
+				y="${chassisWidth}"
+				z="${chassisHeight}"/>
 		</inertial>
 	</link>
@@ -84,5 +78,7 @@
 			<origin xyz="${casterRadius-chassisLength/2} 0 ${casterRadius-chassisHeight+wheelRadius}" rpy="0 0 0"/>
 			<mass value="${casterMass}"/>
-			<sphere_inertia m="${casterMass}" r="${casterRadius}"/>
+			<sphere_inertia
+				m="${casterMass}"
+				r="${casterRadius}"/>
 		</inertial>
 	</link>

Commit message: Change some parameters in my_robot_description

File: my_robot_description/urdf/macros.xacro (robot description, xacro)
@@ -34,5 +34,5 @@
     <link name="${lr}_wheel">
       <collision>
-        <origin xyz="0 0 0" rpy="0 ${PI/2} ${PI/2}" />
+        <origin xyz="0 0 0" rpy="0 ${PI/2} ${PI}" />
         <geometry>
           <cylinder
@@ -42,5 +42,5 @@
       </collision>
       <visual>
-        <origin xyz="0 0 0" rpy="0 ${PI/2} ${PI/2}" />
+        <origin xyz="0 0 0" rpy="0 ${PI/2} ${PI}" />
         <geometry>
           <!--cylinder
@@ -52,5 +52,5 @@
       </visual>
       <inertial>
-        <origin xyz="0 0 0" rpy="0 ${PI/2} ${PI/2}" />
+        <origin xyz="0 0 0" rpy="0 ${PI/2} ${PI}" />
         <mass value="${wheelMass}"/>
         <cylinder_inertia

File: my_robot_description/urdf/my_robot.xacro (robot description, xacro)
@@ -9,9 +9,9 @@
 <robot name="my_robot" xmlns:xacro="http://www.ros.org/wiki/xacro">
 	<xacro:property name="PI" value="3.1415926535897931"/>
-	<xacro:property name="chassisHeight" value="0.037"/>
+	<xacro:property name="chassisHeight" value="0.095"/>
 	<xacro:property name="chassisLength" value="0.175"/>
-	<xacro:property name="chassisWidth" value="0.142"/>
-	<xacro:property name="chassisMass" value="0.25"/>
-	<xacro:property name="casterRadius" value="0.0125"/>
+	<xacro:property name="chassisWidth" value="0.115"/>
+	<xacro:property name="chassisMass" value="0.15"/>
+	<xacro:property name="casterRadius" value="0.015"/>
 	<xacro:property name="casterMass" value="0.05"/>
 	<xacro:property name="wheelWidth" value="0.025"/>
@@ -19,6 +19,6 @@
 	<xacro:property name="wheelPos" value="0.036"/>
 	<xacro:property name="wheelMass" value="0.05"/>
-	<xacro:property name="cameraSize" value="0.05"/>
-	<xacro:property name="cameraMass" value="0.1"/>
+	<!--xacro:property name="cameraSize" value="0.05"/>
+	<xacro:property name="cameraMass" value="0.1"/-->
 	<xacro:include filename="$(find my_robot_description)/urdf/my_robot.gazebo" />
 	<!-- Import Rviz colors -->
@@ -63,10 +63,10 @@
 	</joint>
 	<link name="caster_wheel">
-		<collision>
-			<origin xyz="${casterRadius-chassisLength/2} 0 ${casterRadius-chassisHeight+wheelRadius}" rpy="0 0 0"/>
+		<!--collision>
+			<origin xyz="${casterRadius+chassisLength/2} 0 ${casterRadius-chassisHeight+wheelRadius}" rpy="0 0 0"/>
 			<geometry>
 				<sphere radius="${casterRadius}"/>
 	  		</geometry>
-		</collision>
+		</collision-->
 		<!--visual>
 			<origin xyz="${casterRadius-chassisLength/2} 0 ${casterRadius-chassisHeight+wheelRadius}" rpy="0 0 0"/>
@@ -76,5 +76,5 @@
 		</visual-->
 		<inertial>
-			<origin xyz="${casterRadius-chassisLength/2} 0 ${casterRadius-chassisHeight+wheelRadius}" rpy="0 0 0"/>
+			<origin xyz="${casterRadius+chassisLength/2} 0 ${casterRadius-chassisHeight+wheelRadius}" rpy="0 0 0"/>
 			<mass value="${casterMass}"/>
 			<sphere_inertia
@@ -94,5 +94,7 @@
 			<origin xyz="0 0 0" rpy="0 0 0"/>
 			<geometry>
-				<box size="${cameraSize} ${cameraSize} ${cameraSize}"/>
+				<box size="${cameraSize}
+						   ${cameraSize}
+						   ${cameraSize}"/>
 			</geometry>
 		</collision>
@@ -100,5 +102,7 @@
 			<origin xyz="0 0 0" rpy="0 0 0"/>
 			<geometry>
-				<box size="${cameraSize} ${cameraSize} ${cameraSize}"/>
+				<box size="${cameraSize}
+						   ${cameraSize}
+						   ${cameraSize}"/>
 			</geometry>
 			<material name="blue"/>
@@ -107,5 +111,8 @@
 			<mass value="${cameraMass}" />
 			<origin xyz="0 0 0" rpy="0 0 0"/>
-			<box_inertia m="${cameraMass}" x="${cameraSize}" y="${cameraSize}" z="${cameraSize}" />
+			<box_inertia m="${cameraMass}"
+						 x="${cameraSize}"
+						 y="${cameraSize}"
+						 z="${cameraSize}" />
 		</inertial>
 	</link-->

Commit message: Robot moving wheels but not chassis

File: my_robot_description/urdf/macros.xacro (robot description, xacro)
@@ -3,6 +3,6 @@
 	definitions of some macros for easier description of the robot
 -->
-<robot>
-  <macro name="cylinder_inertia" params="m r h">
+<robot xmlns:xacro="http://www.ros.org/wiki/xacro">
+  <xacro:macro name="cylinder_inertia" params="m r h">
     <inertia  ixx="${m*(3*r*r+h*h)/12}"
     			ixy = "0"
@@ -12,6 +12,6 @@
     			izz="${m*r*r/2}"
     />
-  </macro>
-  <macro name="box_inertia" params="m x y z">
+  </xacro:macro>
+  <xacro:macro name="box_inertia" params="m x y z">
     <inertia  ixx="${m*(y*y+z*z)/12}"
     			ixy = "0"
@@ -21,6 +21,6 @@
     			izz="${m*(x*x+z*z)/12}"
     />
-  </macro>
-  <macro name="sphere_inertia" params="m r">
+  </xacro:macro>
+  <xacro:macro name="sphere_inertia" params="m r">
     <inertia  ixx="${2*m*r*r/5}"
     			ixy = "0"
@@ -30,9 +30,9 @@
     			izz="${2*m*r*r/5}"
     />
-  </macro>
-  <macro name="wheel" params="lr tY">
+  </xacro:macro>
+  <xacro:macro name="wheel" params="lr tY">
     <link name="${lr}_wheel">
       <collision>
-        <origin xyz="0 0 0" rpy="0 ${PI/2} ${PI}" />
+        <origin xyz="0 ${-tY*wheelWidth/6} 0" rpy="0 ${PI/2} ${PI/2}" />
         <geometry>
           <cylinder
@@ -42,5 +42,5 @@
       </collision>
       <visual>
-        <origin xyz="0 0 0" rpy="0 ${PI/2} ${PI}" />
+        <origin xyz="0 ${-tY*wheelWidth/6} 0" rpy="0 ${PI/2} ${PI}" />
         <geometry>
           <!--cylinder
@@ -52,5 +52,5 @@
       </visual>
       <inertial>
-        <origin xyz="0 0 0" rpy="0 ${PI/2} ${PI}" />
+        <origin xyz="0 ${-tY*wheelWidth/6} 0" rpy="0 ${PI/2} ${PI/2}" />
         <mass value="${wheelMass}"/>
         <cylinder_inertia
@@ -66,5 +66,5 @@
       <kd  value="1.0" />
       <fdir1 value="1 0 0"/>
-      <material>Gazebo/Black</material>
+      <material>Gazebo/White</material>
     </gazebo>
     <joint name="${lr}_wheel_hinge" type="continuous">
@@ -72,6 +72,6 @@
       <child link="${lr}_wheel"/>
       <origin
-        xyz = "${+wheelPos-chassisLength/4}
-               ${tY*wheelWidth/2+tY*chassisWidth/2}
+        xyz = "${wheelWidth-chassisLength/4}
+               ${tY*wheelWidth/4+tY*chassisWidth/2}
                ${wheelRadius}"
         rpy = "0 0 0" />
@@ -95,4 +95,4 @@
       </actuator>
     </transmission>
-  </macro>
+  </xacro:macro>
 </robot>

File: my_robot_description/urdf/my_robot.xacro (robot description, xacro)
@@ -9,19 +9,21 @@
 <robot name="my_robot" xmlns:xacro="http://www.ros.org/wiki/xacro">
 	<xacro:property name="PI" value="3.1415926535897931"/>
-	<xacro:property name="chassisHeight" value="0.095"/>
+	<xacro:property name="chassisHeight" value="0.04"/>
 	<xacro:property name="chassisLength" value="0.175"/>
 	<xacro:property name="chassisWidth" value="0.115"/>
 	<xacro:property name="chassisMass" value="0.15"/>
-	<xacro:property name="casterRadius" value="0.015"/>
-	<xacro:property name="casterMass" value="0.05"/>
-	<xacro:property name="wheelWidth" value="0.025"/>
-	<xacro:property name="wheelRadius" value="0.037"/>
-	<xacro:property name="wheelPos" value="0.036"/>
+	<xacro:property name="casterRadius" value="0.005"/>
+	<xacro:property name="casterMass" value="0.09"/>
+	<xacro:property name="wheelWidth" value="0.035"/>
+	<xacro:property name="wheelRadius" value="0.03"/>
+	<!-- offset of the wheel respect to the center of the chassis -->
+	<!--xacro:property name="wheelPos" value="0"/-->
 	<xacro:property name="wheelMass" value="0.05"/>
+	<xacro:property name="wheelOffset" value="0.03"/>
 	<!--xacro:property name="cameraSize" value="0.05"/>
 	<xacro:property name="cameraMass" value="0.1"/-->
-	<xacro:include filename="$(find my_robot_description)/urdf/my_robot.gazebo" />
 	<!-- Import Rviz colors -->
 	<xacro:include filename="$(find my_robot_description)/urdf/materials.xacro" />
+	<xacro:include filename="$(find my_robot_description)/urdf/my_robot.gazebo" />
 	<xacro:include filename="$(find my_robot_description)/urdf/macros.xacro" />
 	<!-- Used for fixing robot to Gazebo 'chassis' -->
@@ -33,13 +35,14 @@
 	<link name='chassis'>
 		<collision>
-			<origin xyz="0 0 ${wheelRadius}" rpy="0 0 0"/>
+			<origin xyz="0 0 ${wheelRadius*2}" rpy="0 0 0"/>
 			<geometry>
-				<box size="${chassisLength}
+				<!--box size="${chassisLength}
 						   ${chassisWidth}
-						   ${chassisHeight}"/>
+						   ${chassisHeight/6}"/-->
+				<mesh filename="package://my_robot_description/meshes/chassis.dae" />
 			</geometry>
 		</collision>
 		<visual>
-			<origin xyz="0 0 ${wheelRadius}" rpy="0 0 0"/>
+			<origin xyz="0 0 ${wheelRadius*2}" rpy="0 0 0"/>
 			<geometry>
 				<!--box size="${chassisLength} ${chassisWidth} ${chassisHeight}"/-->
@@ -49,5 +52,5 @@
 		</visual>
 		<inertial>
-			<origin xyz="0 0 ${wheelRadius}" rpy="0 0 0"/>
+			<origin xyz="0 0 ${wheelRadius*2}" rpy="0 0 0"/>
 			<mass value="${chassisMass}"/>
 			<box_inertia
@@ -55,24 +58,24 @@
 				x="${chassisLength}"
 				y="${chassisWidth}"
-				z="${chassisHeight}"/>
+				z="${chassisHeight/6}"/>
 		</inertial>
 	</link>
-	<joint name="fixed" type="fixed">
+	<!--joint name="fixed" type="fixed">
 		<parent link="chassis"/>
 		<child link="caster_wheel"/>
 	</joint>
 	<link name="caster_wheel">
-		<!--collision>
+		<collision>
 			<origin xyz="${casterRadius+chassisLength/2} 0 ${casterRadius-chassisHeight+wheelRadius}" rpy="0 0 0"/>
 			<geometry>
 				<sphere radius="${casterRadius}"/>
 	  		</geometry>
-		</collision-->
-		<!--visual>
+		</collision>
+		<visual>
 			<origin xyz="${casterRadius-chassisLength/2} 0 ${casterRadius-chassisHeight+wheelRadius}" rpy="0 0 0"/>
 			<geometry>
 				<sphere radius="${casterRadius}"/>
 			</geometry>
-		</visual-->
+		</visual>
 		<inertial>
 			<origin xyz="${casterRadius+chassisLength/2} 0 ${casterRadius-chassisHeight+wheelRadius}" rpy="0 0 0"/>
@@ -82,5 +85,5 @@
 				r="${casterRadius}"/>
 		</inertial>
-	</link>
+	</link-->
 	<wheel lr="left" tY="-1"/>
 	<wheel lr="right" tY="1"/>
