Commit message: Editing Gazebo robot

File: my_robot_description/urdf/macros.xacro (robot description, xacro)
@@ -34,5 +34,6 @@
     <link name="${lr}_wheel">
       <collision>
-        <origin xyz="0 ${-tY*wheelWidth/6} 0" rpy="0 ${PI/2} ${PI/2}" />
+        <origin xyz="0 0 0"
+        		rpy="0 ${PI/2} ${PI/2}" />
         <geometry>
           <cylinder
@@ -42,15 +43,16 @@
       </collision>
       <visual>
-        <origin xyz="0 ${-tY*wheelWidth/6} 0" rpy="0 ${PI/2} ${PI}" />
+        <origin xyz="0 0 0"
+        		rpy="0 ${PI/2} ${PI}" />
         <geometry>
-          <!--cylinder
+          <cylinder
             length="${wheelWidth}"
-            radius="${wheelRadius}"/-->
-          <mesh filename="package://my_robot_description/meshes/${lr}_wheel.dae" />
+            radius="${wheelRadius}"/>
+          <!--mesh filename="package://my_robot_description/meshes/${lr}_wheel.dae" /-->
         </geometry>
-        <material name="black"/>
       </visual>
       <inertial>
-        <origin xyz="0 ${-tY*wheelWidth/6} 0" rpy="0 ${PI/2} ${PI/2}" />
+        <origin xyz="0 0 0"
+        		rpy="0 ${PI/2} ${PI/2}" />
         <mass value="${wheelMass}"/>
         <cylinder_inertia
@@ -72,9 +74,10 @@
       <child link="${lr}_wheel"/>
       <origin
-        xyz = "${wheelWidth-chassisLength/4}
+        xyz = "0
                ${tY*wheelWidth/4+tY*chassisWidth/2}
                ${wheelRadius}"
         rpy = "0 0 0" />
-      <axis xyz="0 1 0" rpy="0 0 0" />
+      <axis xyz="0 1 0"
+      		rpy="0 0 0" />
       <!--limit effort="100" velocity="100"/-->
       <limit effort="10" velocity="10"/>

File: my_robot_description/urdf/my_robot.xacro (robot description, xacro)
@@ -9,16 +9,17 @@
 <robot name="my_robot" xmlns:xacro="http://www.ros.org/wiki/xacro">
 	<xacro:property name="PI" value="3.1415926535897931"/>
-	<xacro:property name="chassisHeight" value="0.04"/>
-	<xacro:property name="chassisLength" value="0.175"/>
-	<xacro:property name="chassisWidth" value="0.115"/>
+	<xacro:property name="chassisHeight" value="0.0623"/>
+	<xacro:property name="chassisLength" value="0.198"/>
+	<xacro:property name="chassisWidth" value="0.119"/>
 	<xacro:property name="chassisMass" value="0.15"/>
-	<xacro:property name="casterRadius" value="0.01"/>
+	<xacro:property name="casterRadius" value="0.0165"/>
 	<xacro:property name="casterMass" value="0.09"/>
-	<xacro:property name="wheelWidth" value="0.035"/>
-	<xacro:property name="wheelRadius" value="0.03"/>
+	<xacro:property name="casterOffsetX" value="0.091"/>
+	<xacro:property name="wheelWidth" value="0.026"/>
+	<xacro:property name="wheelRadius" value="0.032"/>
 	<!-- offset of the wheel respect to the center of the chassis -->
 	<!--xacro:property name="wheelPos" value="0"/-->
 	<xacro:property name="wheelMass" value="0.05"/>
-	<xacro:property name="wheelOffset" value="0.03"/>
+	<xacro:property name="wheelOffsetY" value="-0.047"/>
 	<!--xacro:property name="cameraSize" value="0.05"/>
 	<xacro:property name="cameraMass" value="0.1"/-->
@@ -35,14 +36,14 @@
 	<link name='chassis'>
 		<collision>
-			<origin xyz="0 0 ${wheelRadius+0.05}" rpy="0 0 0"/>
+			<origin xyz="0 0 ${wheelRadius}" rpy="0 0 0"/>
 			<geometry>
-				<!--box size="${chassisLength}
+				<box size="${chassisLength}
 						   ${chassisWidth}
-						   ${chassisHeight}"/-->
-				<mesh filename="package://my_robot_description/meshes/chassis.dae" />
+						   ${chassisHeight}"/>
+				<!--mesh filename="package://my_robot_description/meshes/chassis.dae" /-->
 			</geometry>
 		</collision>
 		<visual>
-			<origin xyz="0 0 ${wheelRadius+0.05}" rpy="0 0 0"/>
+			<origin xyz="0 0 ${wheelRadius}" rpy="0 0 0"/>
 			<geometry>
 				<!--box size="${chassisLength} ${chassisWidth} ${chassisHeight}"/-->
@@ -52,5 +53,5 @@
 		</visual>
 		<inertial>
-			<origin xyz="0 0 ${wheelRadius+0.05}" rpy="0 0 0"/>
+			<origin xyz="0 0 ${wheelRadius}" rpy="0 0 0"/>
 			<mass value="${chassisMass}"/>
 			<box_inertia
@@ -67,5 +68,5 @@
 	<link name="caster_wheel">
 		<collision>
-			<origin xyz="${casterRadius+3*chassisLength/8} 0 ${casterRadius+wheelRadius}" rpy="0 0 0"/>
+			<origin xyz="${casterOffsetX} 0 ${2*casterRadius}" rpy="0 0 0"/>
 			<geometry>
 				<sphere radius="${casterRadius}"/>
@@ -73,5 +74,5 @@
 		</collision>
 		<visual>
-			<origin xyz="${casterRadius+3*chassisLength/8} 0 ${casterRadius+wheelRadius}" rpy="0 0 0"/>
+			<origin xyz="${casterOffsetX} 0 ${2*casterRadius}" rpy="0 0 0"/>
 			<geometry>
 				<!--sphere radius="${casterRadius}"/-->
@@ -81,5 +82,5 @@
 		</visual>
 		<inertial>
-			<origin xyz="${casterRadius+3*chassisLength/8} 0 ${casterRadius+wheelRadius}" rpy="0 0 0"/>
+			<origin xyz="${casterOffsetX} 0 ${2*casterRadius}" rpy="0 0 0"/>
 			<mass value="${casterMass}"/>
 			<sphere_inertia

Commit message: Simplifying model in order to move the robot

File: my_robot_description/urdf/macros.xacro (robot description, xacro)
@@ -35,5 +35,5 @@
       <collision>
         <origin xyz="0 0 0"
-        		rpy="0 ${PI/2} ${PI/2}" />
+        		rpy="0 0 0" />
         <geometry>
           <cylinder
@@ -44,5 +44,5 @@
       <visual>
         <origin xyz="0 0 0"
-        		rpy="0 ${PI/2} ${PI}" />
+        		rpy="0 0 0" />
         <geometry>
           <cylinder
@@ -54,5 +54,5 @@
       <inertial>
         <origin xyz="0 0 0"
-        		rpy="0 ${PI/2} ${PI/2}" />
+        		rpy="0 0 0" />
         <mass value="${wheelMass}"/>
         <cylinder_inertia
@@ -74,12 +74,10 @@
       <child link="${lr}_wheel"/>
       <origin
-        xyz = "0
-               ${tY*wheelWidth/4+tY*chassisWidth/2}
-               ${wheelRadius}"
-        rpy = "0 0 0" />
-      <axis xyz="0 1 0"
+        xyz = "0 ${-tY*(wheelOffsetY+wheelRadius/2)} 0"
+        rpy = "${tY*PI/2} 0 0" />
+      <axis xyz="0 0 1"
       		rpy="0 0 0" />
-      <!--limit effort="100" velocity="100"/-->
-      <limit effort="10" velocity="10"/>
+      <limit effort="100" velocity="100"/>
+      <!--limit effort="10" velocity="10"/-->
       <joint_properties damping="0.0" friction="0.0"/>
     </joint>

File: my_robot_description/urdf/my_robot.xacro (robot description, xacro)
@@ -21,5 +21,5 @@
 	<!--xacro:property name="wheelPos" value="0"/-->
 	<xacro:property name="wheelMass" value="0.05"/>
-	<xacro:property name="wheelOffsetY" value="-0.047"/>
+	<xacro:property name="wheelOffsetY" value="0.047"/>
 	<!--xacro:property name="cameraSize" value="0.05"/>
 	<xacro:property name="cameraMass" value="0.1"/-->
@@ -68,5 +68,6 @@
 	<link name="caster_wheel">
 		<collision>
-			<origin xyz="${casterOffsetX} 0 ${2*casterRadius}" rpy="0 0 0"/>
+			<origin xyz="${casterOffsetX} 0 ${casterRadius}"
+					rpy="0 0 0"/>
 			<geometry>
 				<sphere radius="${casterRadius}"/>
@@ -74,13 +75,15 @@
 		</collision>
 		<visual>
-			<origin xyz="${casterOffsetX} 0 ${2*casterRadius}" rpy="0 0 0"/>
+			<origin xyz="${casterOffsetX} 0 ${casterRadius}"
+					rpy="0 0 0"/>
 			<geometry>
-				<!--sphere radius="${casterRadius}"/-->
-				<mesh filename="package://my_robot_description/meshes/caster_wheel.dae" />
+				<sphere radius="${2*casterRadius}"/>
+				<!--mesh filename="package://my_robot_description/meshes/caster_wheel.dae" /-->
 			</geometry>
 			<material name="grey" />
 		</visual>
 		<inertial>
-			<origin xyz="${casterOffsetX} 0 ${2*casterRadius}" rpy="0 0 0"/>
+			<origin xyz="${casterOffsetX} 0 ${casterRadius}"
+					rpy="0 0 0"/>
 			<mass value="${casterMass}"/>
 			<sphere_inertia

Commit message: Continue editing

File: my_robot_description/urdf/macros.xacro (robot description, xacro)
@@ -73,7 +73,10 @@
       <parent link="chassis"/>
       <child link="${lr}_wheel"/>
+      <!--origin
+        xyz = "0 ${-tY*(wheelOffsetY+wheelRadius/2)} 0"
+        rpy = "${tY*PI/2} 0 0" /-->
       <origin
-        xyz = "0 ${-tY*(wheelOffsetY+wheelRadius/2)} 0"
-        rpy = "${tY*PI/2} 0 0" />
+      	xyz = "0 ${-tY*chassisWidth/2} 0"
+      	rpy = "${tY*PI/2} 0 0" />
       <axis xyz="0 0 1"
       		rpy="0 0 0" />

File: my_robot_description/urdf/my_robot.xacro (robot description, xacro)
@@ -9,5 +9,6 @@
 <robot name="my_robot" xmlns:xacro="http://www.ros.org/wiki/xacro">
 	<xacro:property name="PI" value="3.1415926535897931"/>
-	<xacro:property name="chassisHeight" value="0.0623"/>
+	<!--xacro:property name="chassisHeight" value="0.0623"/-->
+	<xacro:property name="chassisHeight" value="0.02" />
 	<xacro:property name="chassisLength" value="0.198"/>
 	<xacro:property name="chassisWidth" value="0.119"/>
@@ -18,6 +19,4 @@
 	<xacro:property name="wheelWidth" value="0.026"/>
 	<xacro:property name="wheelRadius" value="0.032"/>
-	<!-- offset of the wheel respect to the center of the chassis -->
-	<!--xacro:property name="wheelPos" value="0"/-->
 	<xacro:property name="wheelMass" value="0.05"/>
 	<xacro:property name="wheelOffsetY" value="0.047"/>
@@ -35,5 +34,5 @@
 	</joint>
 	<link name='chassis'>
-		<collision>
+		<collision name="chassis_collision">
 			<origin xyz="0 0 ${wheelRadius}" rpy="0 0 0"/>
 			<geometry>
@@ -44,13 +43,13 @@
 			</geometry>
 		</collision>
-		<visual>
+		<visual name="chassis_visual">
 			<origin xyz="0 0 ${wheelRadius}" rpy="0 0 0"/>
 			<geometry>
-				<!--box size="${chassisLength} ${chassisWidth} ${chassisHeight}"/-->
-				<mesh filename="package://my_robot_description/meshes/chassis.dae" />
+				<box size="${chassisLength} ${chassisWidth} ${chassisHeight}"/>
+				<!--mesh filename="package://my_robot_description/meshes/chassis.dae" /-->
 			</geometry>
 			<material name="red"/>
 		</visual>
-		<inertial>
+		<inertial name="chassis_inertia">
 			<origin xyz="0 0 ${wheelRadius}" rpy="0 0 0"/>
 			<mass value="${chassisMass}"/>
@@ -61,12 +60,6 @@
 				z="${chassisHeight}"/>
 		</inertial>
-	</link>
-	<joint name="fixed" type="fixed">
-		<parent link="chassis"/>
-		<child link="caster_wheel"/>
-	</joint>
-	<link name="caster_wheel">
-		<collision>
-			<origin xyz="${casterOffsetX} 0 ${casterRadius}"
+		<collision name="caster_collision">
+			<origin xyz="${casterOffsetX} 0 0"
 					rpy="0 0 0"/>
 			<geometry>
@@ -74,15 +67,15 @@
 	  		</geometry>
 		</collision>
-		<visual>
-			<origin xyz="${casterOffsetX} 0 ${casterRadius}"
+		<visual name="caster_visual">
+			<origin xyz="${casterOffsetX} 0 0"
 					rpy="0 0 0"/>
 			<geometry>
-				<sphere radius="${2*casterRadius}"/>
+				<sphere radius="${casterRadius}"/>
 				<!--mesh filename="package://my_robot_description/meshes/caster_wheel.dae" /-->
 			</geometry>
 			<material name="grey" />
 		</visual>
-		<inertial>
-			<origin xyz="${casterOffsetX} 0 ${casterRadius}"
+		<inertial name="caster_inertia">
+			<origin xyz="${casterOffsetX} 0 0"
 					rpy="0 0 0"/>
 			<mass value="${casterMass}"/>

Commit message: Robot won't move

File: my_robot_description/urdf/macros.xacro (robot description, xacro)
@@ -35,14 +35,5 @@
       <collision>
         <origin xyz="0 0 0"
-        		rpy="0 0 0" />
-        <geometry>
-          <cylinder
-            length="${wheelWidth}"
-            radius="${wheelRadius}"/>
-        </geometry>
-      </collision>
-      <visual>
-        <origin xyz="0 0 0"
-        		rpy="0 0 0" />
+        		rpy="${-tY*PI/2} 0 0" />
         <geometry>
           <cylinder
@@ -51,8 +42,18 @@
           <!--mesh filename="package://my_robot_description/meshes/${lr}_wheel.dae" /-->
         </geometry>
+      </collision>
+      <visual>
+        <origin xyz="0 0 0"
+        		rpy="${-tY*PI/2} 0 0" />
+        <geometry>
+          <!--cylinder
+            length="${wheelWidth}"
+            radius="${wheelRadius}"/-->
+          <mesh filename="package://my_robot_description/meshes/${lr}_wheel.dae" />
+        </geometry>
       </visual>
       <inertial>
         <origin xyz="0 0 0"
-        		rpy="0 0 0" />
+        		rpy="${-tY*PI/2} 0 0" />
         <mass value="${wheelMass}"/>
         <cylinder_inertia
@@ -73,13 +74,10 @@
       <parent link="chassis"/>
       <child link="${lr}_wheel"/>
-      <!--origin
-        xyz = "0 ${-tY*(wheelOffsetY+wheelRadius/2)} 0"
-        rpy = "${tY*PI/2} 0 0" /-->
       <origin
-      	xyz = "0 ${-tY*chassisWidth/2} 0"
-      	rpy = "${tY*PI/2} 0 0" />
-      <axis xyz="0 0 1"
-      		rpy="0 0 0" />
-      <limit effort="100" velocity="100"/>
+        xyz = "0 ${-tY*(wheelOffsetY+wheelRadius/2)} ${wheelRadius}"
+        rpy = "0 0 0" />
+      <axis xyz="0 1 0"
+      		  rpy="0 0 0" />
+      <limit effort="100" velocity="10"/>
       <!--limit effort="10" velocity="10"/-->
       <joint_properties damping="0.0" friction="0.0"/>
@@ -95,6 +93,6 @@
       <actuator name="${lr}Motor">
         <hardwareInterface>hardware_interface/EffortJointInterface</hardwareInterface>
-        <!--mechanicalReduction>10</mechanicalReduction-->
-        <mechanicalReduction>1</mechanicalReduction>
+        <mechanicalReduction>10</mechanicalReduction>
+        <!--mechanicalReduction>1</mechanicalReduction-->
       </actuator>
     </transmission>

File: my_robot_description/urdf/materials.xacro (robot description, xacro)
@@ -16,4 +16,10 @@
 	  <color rgba="0.2 0.2 0.2 1.0"/>
 	</material>
+	<material name="light_grey">
+      <color rgba="0.6 0.6 0.6 1"/>
+    </material>
+    <material name="dark_grey">
+      <color rgba="0.3 0.3 0.3 1"/>
+    </material>
 	<material name="orange">
 	  <color rgba="${255/255} ${108/255} ${10/255} 1.0"/>

File: my_robot_description/urdf/my_robot.xacro (robot description, xacro)
@@ -4,23 +4,10 @@
 	#######################################################
     To run:
-    $ roslaunch my_robot_gazebo my_robot_world.launch
+    $ roslaunch my_robot_gazebo my_robot_world.launch paused:=true
     $ rosrun turtlebot_teleop turtlebot_teleop_key /turtlebot_teleop/cmd_vel:=/my_robot/cmd_vel
 -->
 <robot name="my_robot" xmlns:xacro="http://www.ros.org/wiki/xacro">
-	<xacro:property name="PI" value="3.1415926535897931"/>
-	<!--xacro:property name="chassisHeight" value="0.0623"/-->
-	<xacro:property name="chassisHeight" value="0.02" />
-	<xacro:property name="chassisLength" value="0.198"/>
-	<xacro:property name="chassisWidth" value="0.119"/>
-	<xacro:property name="chassisMass" value="0.15"/>
-	<xacro:property name="casterRadius" value="0.0165"/>
-	<xacro:property name="casterMass" value="0.09"/>
-	<xacro:property name="casterOffsetX" value="0.091"/>
-	<xacro:property name="wheelWidth" value="0.026"/>
-	<xacro:property name="wheelRadius" value="0.032"/>
-	<xacro:property name="wheelMass" value="0.05"/>
-	<xacro:property name="wheelOffsetY" value="0.047"/>
-	<!--xacro:property name="cameraSize" value="0.05"/>
-	<xacro:property name="cameraMass" value="0.1"/-->
+	<!-- Robot constants and properties -->
+	<xacro:include filename="$(find my_robot_description)/urdf/my_robot_properties.xacro" />
 	<!-- Import Rviz colors -->
 	<xacro:include filename="$(find my_robot_description)/urdf/materials.xacro" />
@@ -34,23 +21,25 @@
 	</joint>
 	<link name='chassis'>
-		<collision name="chassis_collision">
-			<origin xyz="0 0 ${wheelRadius}" rpy="0 0 0"/>
+		<collision>
+			<origin xyz="0 0 ${wheelRadius}"
+					rpy="0 ${robotPitchAngle} 0"/>
 			<geometry>
-				<box size="${chassisLength}
+				<!--box size="${chassisLength}
 						   ${chassisWidth}
-						   ${chassisHeight}"/>
-				<!--mesh filename="package://my_robot_description/meshes/chassis.dae" /-->
+						   ${chassisHeight}"/-->
+				<mesh filename="package://my_robot_description/meshes/chassis.dae" />
 			</geometry>
 		</collision>
-		<visual name="chassis_visual">
-			<origin xyz="0 0 ${wheelRadius}" rpy="0 0 0"/>
+		<visual>
+			<origin xyz="0 0 ${wheelRadius}"
+					rpy="0 ${robotPitchAngle} 0"/>
 			<geometry>
-				<box size="${chassisLength} ${chassisWidth} ${chassisHeight}"/>
-				<!--mesh filename="package://my_robot_description/meshes/chassis.dae" /-->
+				<mesh filename="package://my_robot_description/meshes/chassis.dae" />
 			</geometry>
 			<material name="red"/>
 		</visual>
-		<inertial name="chassis_inertia">
-			<origin xyz="0 0 ${wheelRadius}" rpy="0 0 0"/>
+		<inertial>
+			<origin xyz="0 0 ${wheelRadius}"
+					rpy="0 ${robotPitchAngle} 0"/>
 			<mass value="${chassisMass}"/>
 			<box_inertia
@@ -60,14 +49,21 @@
 				z="${chassisHeight}"/>
 		</inertial>
-		<collision name="caster_collision">
-			<origin xyz="${casterOffsetX} 0 0"
-					rpy="0 0 0"/>
+	</link>
+	<joint name="caster_joint" type="fixed">
+		<parent link="chassis"/>
+		<child link="caster_wheel"/>
+	</joint>
+	<link name="caster_wheel">
+		<collision>
+			<origin xyz="${casterOffsetX} 0 ${casterRadius}"
+					rpy="0 ${robotPitchAngle} 0"/>
 			<geometry>
 				<sphere radius="${casterRadius}"/>
+				<!--mesh filename="package://my_robot_description/meshes/caster_wheel.dae" /-->
 	  		</geometry>
 		</collision>
-		<visual name="caster_visual">
-			<origin xyz="${casterOffsetX} 0 0"
-					rpy="0 0 0"/>
+		<visual>
+			<origin xyz="${casterOffsetX} 0 ${casterRadius}"
+					rpy="0 ${robotPitchAngle} 0"/>
 			<geometry>
 				<sphere radius="${casterRadius}"/>
@@ -76,7 +72,7 @@
 			<material name="grey" />
 		</visual>
-		<inertial name="caster_inertia">
-			<origin xyz="${casterOffsetX} 0 0"
-					rpy="0 0 0"/>
+		<inertial>
+			<origin xyz="${casterOffsetX} 0 ${casterRadius}"
+					rpy="0 ${robotPitchAngle} 0"/>
 			<mass value="${casterMass}"/>
 			<sphere_inertia

Commit message: It works!

File: my_robot_description/urdf/macros.xacro (robot description, xacro)
@@ -67,6 +67,9 @@
       <mu2 value="1.0"/>
       <kp  value="10000000.0" />
-      <kd  value="1.0" />
-      <fdir1 value="1 0 0"/>
+      <kd>100.0</kd>
+      <minDepth>0.001</minDepth>
+      <maxVel>1.0</maxVel>
+      <!--kd  value="1.0" />
+      <fdir1 value="1 0 0"/-->
       <material>Gazebo/White</material>
     </gazebo>
@@ -79,6 +82,6 @@
       <axis xyz="0 1 0"
       		  rpy="0 0 0" />
-      <limit effort="100" velocity="10"/>
-      <!--limit effort="10" velocity="10"/-->
+      <!--limit effort="100" velocity="10"/-->
+      <limit effort="0.0" velocity="0.0"/>
       <joint_properties damping="0.0" friction="0.0"/>
     </joint>

File: my_robot_description/urdf/my_robot.xacro (robot description, xacro)
@@ -15,7 +15,7 @@
 	<xacro:include filename="$(find my_robot_description)/urdf/macros.xacro" />
 	<!-- Used for fixing robot to Gazebo 'chassis' -->
-	<link name="world" />
+	<link name="base_footprint" />
 	<joint name="base_joint" type="fixed">
-		<parent link="world"/>
+		<parent link="base_footprint"/>
 		<child link="chassis"/>
 	</joint>

Commit message: Change some visual aspects

File: my_robot_description/urdf/macros.xacro (robot description, xacro)
@@ -72,5 +72,5 @@
       <!--kd  value="1.0" />
       <fdir1 value="1 0 0"/-->
-      <material>Gazebo/White</material>
+      <material>Gazebo/FlatBlack</material>
     </gazebo>
     <joint name="${lr}_wheel_hinge" type="continuous">

File: my_robot_description/urdf/my_robot.xacro (robot description, xacro)
@@ -23,5 +23,5 @@
 		<collision>
 			<origin xyz="0 0 ${wheelRadius}"
-					rpy="0 ${robotPitchAngle} 0"/>
+					rpy="0 0 0"/>
 			<geometry>
 				<!--box size="${chassisLength}
@@ -33,5 +33,5 @@
 		<visual>
 			<origin xyz="0 0 ${wheelRadius}"
-					rpy="0 ${robotPitchAngle} 0"/>
+					rpy="0 0 0"/>
 			<geometry>
 				<mesh filename="package://my_robot_description/meshes/chassis.dae" />
@@ -41,5 +41,5 @@
 		<inertial>
 			<origin xyz="0 0 ${wheelRadius}"
-					rpy="0 ${robotPitchAngle} 0"/>
+					rpy="0 0 0"/>
 			<mass value="${chassisMass}"/>
 			<box_inertia
@@ -56,23 +56,23 @@
 	<link name="caster_wheel">
 		<collision>
-			<origin xyz="${casterOffsetX} 0 ${casterRadius}"
-					rpy="0 ${robotPitchAngle} 0"/>
+			<origin xyz="${casterOffsetX} 0 ${2*casterRadius}"
+					rpy="0 0 0"/>
 			<geometry>
-				<sphere radius="${casterRadius}"/>
-				<!--mesh filename="package://my_robot_description/meshes/caster_wheel.dae" /-->
+				<!--sphere radius="${casterRadius}"/-->
+				<mesh filename="package://my_robot_description/meshes/caster_wheel.dae" />
 	  		</geometry>
 		</collision>
 		<visual>
-			<origin xyz="${casterOffsetX} 0 ${casterRadius}"
-					rpy="0 ${robotPitchAngle} 0"/>
+			<origin xyz="${casterOffsetX} 0 ${2*casterRadius}"
+					rpy="0 0 0"/>
 			<geometry>
-				<sphere radius="${casterRadius}"/>
-				<!--mesh filename="package://my_robot_description/meshes/caster_wheel.dae" /-->
+				<!--sphere radius="${casterRadius}"/-->
+				<mesh filename="package://my_robot_description/meshes/caster_wheel.dae" />
 			</geometry>
 			<material name="grey" />
 		</visual>
 		<inertial>
-			<origin xyz="${casterOffsetX} 0 ${casterRadius}"
-					rpy="0 ${robotPitchAngle} 0"/>
+			<origin xyz="${casterOffsetX} 0 ${2*casterRadius}"
+					rpy="0 0 0"/>
 			<mass value="${casterMass}"/>
 			<sphere_inertia

File: my_robot_description/urdf/my_robot_properties.xacro (robot description, xacro)
@@ -6,6 +6,5 @@
 	<xacro:property name="chassisWidth" value="0.119"/>
 	<xacro:property name="chassisMass" value="0.15"/>
-	<!--xacro:property name="casterRadius" value="0.0165"/-->
-	<xacro:property name="casterRadius" value="0.022"/>
+	<xacro:property name="casterRadius" value="0.021"/>
 	<xacro:property name="casterMass" value="0.09"/>
 	<xacro:property name="casterOffsetX" value="0.091"/>
@@ -14,5 +13,4 @@
 	<xacro:property name="wheelMass" value="0.05"/>
 	<xacro:property name="wheelOffsetY" value="0.047"/>
-	<xacro:property name="robotPitchAngle" value="0"/>
 	<!--xacro:property name="cameraSize" value="0.05"/>
 	<xacro:property name="cameraMass" value="0.1"/-->
