Commit message: Edit some params and add links for reference

File: my_robot_description/urdf/macros.xacro (robot description, xacro)
@@ -43,5 +43,4 @@
             length="${wheelWidth}"
             radius="${wheelRadius}"/>
-          <!--mesh filename="package://my_robot_description/meshes/${lr}_wheel.dae" /-->
         </geometry>
       </collision>
@@ -50,7 +49,4 @@
         		rpy="${-tY*PI/2} 0 0" />
         <geometry>
-          <!--cylinder
-            length="${wheelWidth}"
-            radius="${wheelRadius}"/-->
           <mesh filename="package://my_robot_description/meshes/${lr}_wheel.dae" />
         </geometry>
@@ -81,5 +77,5 @@
       <child link="${lr}_wheel"/>
       <origin
-        xyz = "0 ${-tY*(wheelOffsetY+wheelRadius/2)} ${wheelRadius}"
+        xyz = "0 ${-tY*(wheelOffsetY+wheelWidth)} ${wheelRadius}"
         rpy = "0 0 0" />
       <axis xyz="0 1 0"

File: my_robot_description/urdf/my_robot.xacro (robot description, xacro)
@@ -15,5 +15,5 @@
 	<xacro:include filename="$(find my_robot_description)/urdf/my_robot.gazebo" />
 	<!-- Inertia matrices -->
-	<xacro:include filename="$(find my_robot_description)/urdf/inertias.xacro" />
+	<xacro:include filename="$(find my_robot_description)/urdf/macros.xacro" />
 	<!-- Used for fixing robot to Gazebo 'chassis' -->
 	<link name="base_footprint" />

File: my_robot_description/urdf/my_robot_properties.xacro (robot description, xacro)
@@ -16,5 +16,5 @@
 	<xacro:property name="wheelRadius" value="0.032"/>
 	<xacro:property name="wheelMass" value="0.05"/>
-	<xacro:property name="wheelOffsetY" value="0.047"/>
+	<xacro:property name="wheelOffsetY" value="0.037"/>
 	<!-- Velodyne properties -->
 	<xacro:property name="velodyneLengthBottom" value="0.05867"/>

File: my_robot_description/urdf/velodyne.xacro (robot description, xacro)
@@ -5,4 +5,7 @@
   http://gazebosim.org/tutorials?cat=guided_i&tut=guided_i1
   http://gazebosim.org/tutorials
+  Another approach:
+    https://github.com/richardw05/mybot_ws/tree/master/src
+    Nav: http://moorerobots.com/blog/post/3
 -->
 <robot xmlns:xacro="http://www.ros.org/wiki/xacro">
@@ -10,5 +13,5 @@
   <xacro:include filename="$(find my_robot_description)/urdf/my_robot_properties.xacro" />
   <!-- Inertia matrices -->
-  <xacro:include filename="$(find my_robot_description)/urdf/inertias.xacro" />
+  <xacro:include filename="$(find my_robot_description)/urdf/macros.xacro" />
   <joint name="robot_to_velodyne_joint" type="fixed">
     <origin xyz="${-velodyneLengthBottom+chassisLength/2}
@@ -30,5 +33,5 @@
         h="${velodyneLengthBottom}" />
     </inertial>
-    <collision name="vbase_collision">
+    <collision name="velodyne_bottom_collision">
       <geometry>
         <!-- Radius and length provided by Velodyne -->
@@ -38,5 +41,5 @@
     </collision>
     <!-- The visual is mostly a copy of the collision -->
-    <visual name="vbase_visual">
+    <visual name="velodyne_bottom_visual">
       <geometry>
         <cylinder length="${velodyneLengthBottom}"
