Commit message: Add a caster wheel as a separate mesh

File: my_robot_description/urdf/my_robot.xacro (robot description, xacro)
@@ -13,5 +13,5 @@
 	<xacro:property name="chassisWidth" value="0.115"/>
 	<xacro:property name="chassisMass" value="0.15"/>
-	<xacro:property name="casterRadius" value="0.005"/>
+	<xacro:property name="casterRadius" value="0.01"/>
 	<xacro:property name="casterMass" value="0.09"/>
 	<xacro:property name="wheelWidth" value="0.035"/>
@@ -35,14 +35,14 @@
 	<link name='chassis'>
 		<collision>
-			<origin xyz="0 0 ${wheelRadius*2}" rpy="0 0 0"/>
+			<origin xyz="0 0 ${wheelRadius+0.05}" rpy="0 0 0"/>
 			<geometry>
 				<!--box size="${chassisLength}
 						   ${chassisWidth}
-						   ${chassisHeight/6}"/-->
+						   ${chassisHeight}"/-->
 				<mesh filename="package://my_robot_description/meshes/chassis.dae" />
 			</geometry>
 		</collision>
 		<visual>
-			<origin xyz="0 0 ${wheelRadius*2}" rpy="0 0 0"/>
+			<origin xyz="0 0 ${wheelRadius+0.05}" rpy="0 0 0"/>
 			<geometry>
 				<!--box size="${chassisLength} ${chassisWidth} ${chassisHeight}"/-->
@@ -52,5 +52,5 @@
 		</visual>
 		<inertial>
-			<origin xyz="0 0 ${wheelRadius*2}" rpy="0 0 0"/>
+			<origin xyz="0 0 ${wheelRadius+0.05}" rpy="0 0 0"/>
 			<mass value="${chassisMass}"/>
 			<box_inertia
@@ -58,8 +58,8 @@
 				x="${chassisLength}"
 				y="${chassisWidth}"
-				z="${chassisHeight/6}"/>
+				z="${chassisHeight}"/>
 		</inertial>
 	</link>
-	<!--joint name="fixed" type="fixed">
+	<joint name="fixed" type="fixed">
 		<parent link="chassis"/>
 		<child link="caster_wheel"/>
@@ -67,5 +67,5 @@
 	<link name="caster_wheel">
 		<collision>
-			<origin xyz="${casterRadius+chassisLength/2} 0 ${casterRadius-chassisHeight+wheelRadius}" rpy="0 0 0"/>
+			<origin xyz="${casterRadius+3*chassisLength/8} 0 ${casterRadius+wheelRadius}" rpy="0 0 0"/>
 			<geometry>
 				<sphere radius="${casterRadius}"/>
@@ -73,11 +73,13 @@
 		</collision>
 		<visual>
-			<origin xyz="${casterRadius-chassisLength/2} 0 ${casterRadius-chassisHeight+wheelRadius}" rpy="0 0 0"/>
+			<origin xyz="${casterRadius+3*chassisLength/8} 0 ${casterRadius+wheelRadius}" rpy="0 0 0"/>
 			<geometry>
-				<sphere radius="${casterRadius}"/>
+				<!--sphere radius="${casterRadius}"/-->
+				<mesh filename="package://my_robot_description/meshes/caster_wheel.dae" />
 			</geometry>
+			<material name="grey" />
 		</visual>
 		<inertial>
-			<origin xyz="${casterRadius+chassisLength/2} 0 ${casterRadius-chassisHeight+wheelRadius}" rpy="0 0 0"/>
+			<origin xyz="${casterRadius+3*chassisLength/8} 0 ${casterRadius+wheelRadius}" rpy="0 0 0"/>
 			<mass value="${casterMass}"/>
 			<sphere_inertia
@@ -85,5 +87,5 @@
 				r="${casterRadius}"/>
 		</inertial>
-	</link-->
+	</link>
 	<wheel lr="left" tY="-1"/>
 	<wheel lr="right" tY="1"/>

Commit message: Add Hokuyo laser

File: my_robot_description/urdf/my_robot.xacro (robot description, xacro)
@@ -80,7 +80,5 @@
 	<wheel lr="left" tY="-1"/>
 	<wheel lr="right" tY="1"/>
-	<!-- Including Velodyne model -->
-	<xacro:include filename="$(find my_robot_description)/urdf/velodyne.xacro" />
-	<!-- Camera model -->
-	<!--xacro:include filename="$(find my_robot_description)/urdf/camera.xacro" /-->
+	<!-- Sensor models -->
+	<xacro:include filename="$(find my_robot_description)/urdf/sensors.xacro" />
 </robot>

File: my_robot_description/urdf/my_robot_properties.xacro (robot description, xacro)
@@ -17,12 +17,12 @@
 	<xacro:property name="wheelMass" value="0.05"/>
 	<xacro:property name="wheelOffsetY" value="0.037"/>
-	<!-- Velodyne properties -->
-	<xacro:property name="velodyneLengthBottom" value="0.05867"/>
-	<xacro:property name="velodyneLengthTop" value="0.07357"/>
-	<xacro:property name="velodyneMassBottom" value="1.2"/>
-	<xacro:property name="velodyneMassTop" value="0.1"/>
-	<xacro:property name="velodyneRadius" value="0.04267"/>
+	<!-- Hokuyo laser properties -->
+	<xacro:property name="hokuyoMass" value="1e-5"/>
+	<xacro:property name="hokuyoLength" value="0.1"/>
+	<xacro:property name="hokuyoWidth" value="0.1"/>
+	<xacro:property name="hokuyoHeight" value="0.1"/>
+	<xacro:property name="hokuyoOffsetZ" value="0.1"/>
 	<!-- Camera properties -->
 	<xacro:property name="cameraSize" value="0.05"/>
-	<xacro:property name="cameraMass" value="0.1"/>
+	<xacro:property name="cameraMass" value="0.9"/>
 </robot>
