Commit message: Testing Hokuyo model in Gazebo

File: my_robot_description/urdf/sensors.xacro (robot description, xacro)
@@ -55,8 +55,8 @@
             rpy="0 0 0"/>
     <parent link="chassis"/>
-    <child link="hokuyo"/>
+    <child link="hokuyo_link"/>
   </joint>
   <!-- Hokuyo Laser -->
-  <link name="hokuyo">
+  <link name="hokuyo_link">
     <collision>
       <origin xyz="0 0 0"
@@ -83,4 +83,6 @@
         z="${hokuyoHeight}"/>
     </inertial>
+    <!-- Gazebo plugin -->
+    <!--my_robot_sim_laser_range_finder/-->
   </link>
 </robot>

Commit message: New changes

File: my_robot_description/urdf/sensors.xacro (robot description, xacro)
@@ -13,5 +13,5 @@
   <!-- Inertia matrices -->
   <xacro:include filename="$(find my_robot_description)/urdf/macros.xacro" />
-  <link name="camera">
+  <link name="camera_link">
     <collision>
       <origin xyz="0 0 0"
@@ -42,4 +42,6 @@
                    z="${cameraSize}" />
     </inertial>
+    <!-- Gazebo plugin -->
+    <my_robot_sim_camera/>
   </link>
   <joint name="camera_joint" type="fixed">
@@ -48,5 +50,5 @@
             rpy="0 0 0"/>
     <parent link="chassis"/>
-    <child link="camera"/>
+    <child link="camera_link"/>
   </joint>
   <joint name="hokuyo_joint" type="fixed">
@@ -84,5 +86,5 @@
     </inertial>
     <!-- Gazebo plugin -->
-    <!--my_robot_sim_laser_range_finder/-->
+    <my_robot_sim_laser_range_finder/>
   </link>
 </robot>

Commit message: more testing with Hokuyo

File: my_robot_description/urdf/sensors.xacro (robot description, xacro)
@@ -13,4 +13,6 @@
   <!-- Inertia matrices -->
   <xacro:include filename="$(find my_robot_description)/urdf/macros.xacro" />
+  <!-- Gazebo aspects of the robot -->
+  <xacro:include filename="$(find my_robot_description)/urdf/my_robot.gazebo" />
   <link name="camera_link">
     <collision>
@@ -42,6 +44,4 @@
                    z="${cameraSize}" />
     </inertial>
-    <!-- Gazebo plugin -->
-    <my_robot_sim_camera/>
   </link>
   <joint name="camera_joint" type="fixed">
@@ -71,5 +71,6 @@
     </collision>
     <visual>
-      <origin xyz="0 0 0" rpy="0 0 0"/>
+      <origin xyz="0 0 0"
+              rpy="0 0 0"/>
       <geometry>
         <mesh filename="package://my_robot_description/meshes/hokuyo.dae"/>
@@ -78,5 +79,6 @@
     <inertial>
       <mass value="${hokuyoMass}" />
-      <origin xyz="0 0 0" rpy="0 0 0"/>
+      <origin xyz="0 0 0"
+              rpy="0 0 0"/>
       <box_inertia
         m="${hokuyoMass}"
@@ -85,6 +87,4 @@
         z="${hokuyoHeight}"/>
     </inertial>
-    <!-- Gazebo plugin -->
-    <my_robot_sim_laser_range_finder/>
   </link>
 </robot>
