Commit message: RViz changes in robot model

File: my_robot_description/urdf/my_robot_properties.xacro (robot description, xacro)
@@ -19,10 +19,11 @@
 	<!-- Hokuyo laser properties -->
 	<xacro:property name="hokuyoMass" value="1e-5"/>
-	<xacro:property name="hokuyoLength" value="0.1"/>
-	<xacro:property name="hokuyoWidth" value="0.1"/>
-	<xacro:property name="hokuyoHeight" value="0.1"/>
-	<xacro:property name="hokuyoOffsetZ" value="0.1"/>
+	<xacro:property name="hokuyoLength" value="0.05"/>
+	<xacro:property name="hokuyoWidth" value="0.05"/>
+	<xacro:property name="hokuyoHeight" value="0.07"/>
+	<xacro:property name="hokuyoOffsetZ" value="0.1125"/>
 	<!-- Camera properties -->
 	<xacro:property name="cameraSize" value="0.05"/>
 	<xacro:property name="cameraMass" value="0.9"/>
+	<xacro:property name="cameraOffsetX" value="0.095"/>
 </robot>

File: my_robot_description/urdf/sensors.xacro (robot description, xacro)
@@ -4,7 +4,4 @@
   http://moorerobots.com/blog/post/3
   https://github.com/richardw05/mybot_ws/tree/master/src
-  https://github.com/richardw05/mybot_ws/blob/master/src/mybot_description/launch/mybot_rviz.launch
-  https://github.com/richardw05/mybot_ws/blob/master/src/mybot_description/launch/mybot_rviz_amcl.launch
-  https://github.com/richardw05/mybot_ws/blob/master/src/mybot_description/launch/mybot_rviz_gmapping.launch
 -->
 <robot xmlns:xacro="http://www.ros.org/wiki/xacro">
@@ -13,7 +10,45 @@
   <!-- Inertia matrices -->
   <xacro:include filename="$(find my_robot_description)/urdf/macros.xacro" />
+  <link name="camera">
+    <collision>
+      <origin xyz="0 0 0"
+              rpy="0 0 0"/>
+      <geometry>
+        <box size="${cameraSize}
+                   ${cameraSize}
+                   ${cameraSize}"/>
+      </geometry>
+    </collision>
+    <visual>
+      <origin xyz="0 0 0"
+              rpy="0 0 0"/>
+      <geometry>
+        <box size="${cameraSize}
+                   ${cameraSize}
+                   ${cameraSize}"/>
+      </geometry>
+      <material name="green"/>
+    </visual>
+    <inertial>
+      <mass value="${cameraMass}" />
+      <origin xyz="0 0 0"
+              rpy="0 0 0"/>
+      <box_inertia m="${cameraMass}"
+                   x="${cameraSize}"
+                   y="${cameraSize}"
+                   z="${cameraSize}" />
+    </inertial>
+  </link>
+  <joint name="camera_joint" type="fixed">
+    <axis xyz="0 1 0" />
+    <origin xyz="${cameraOffsetX} 0 ${2*wheelRadius}"
+            rpy="0 0 0"/>
+    <parent link="chassis"/>
+    <child link="camera"/>
+  </joint>
   <joint name="hokuyo_joint" type="fixed">
     <axis xyz="0 1 0" />
-    <origin xyz="${casterOffsetX} 0 ${hokuyoOffsetZ}" rpy="0 0 0"/>
+    <origin xyz="0 0 ${hokuyoOffsetZ}"
+            rpy="0 0 0"/>
     <parent link="chassis"/>
     <child link="hokuyo"/>
@@ -25,8 +60,7 @@
               rpy="0 0 0"/>
       <geometry>
-        <box size="
-          ${hokuyoLength}
-          ${hokuyoWidth}
-          ${hokuyoHeight}"/>
+        <box size="${hokuyoLength}
+                   ${hokuyoWidth}
+                   ${hokuyoHeight}"/>
       </geometry>
     </collision>

Commit message: Change camera mass

File: my_robot_description/urdf/my_robot_properties.xacro (robot description, xacro)
@@ -25,5 +25,5 @@
 	<!-- Camera properties -->
 	<xacro:property name="cameraSize" value="0.05"/>
-	<xacro:property name="cameraMass" value="0.9"/>
+	<xacro:property name="cameraMass" value="0.05"/>
 	<xacro:property name="cameraOffsetX" value="0.095"/>
 </robot>

Commit message: Edit camera size and location

File: my_robot_description/urdf/my_robot_properties.xacro (robot description, xacro)
@@ -24,6 +24,9 @@
 	<xacro:property name="hokuyoOffsetZ" value="0.1125"/>
 	<!-- Camera properties -->
-	<xacro:property name="cameraSize" value="0.05"/>
+	<xacro:property name="cameraLength" value="0.04"/>
+	<xacro:property name="cameraWidth" value="0.08"/>
+	<xacro:property name="cameraHeight" value="0.03"/>
 	<xacro:property name="cameraMass" value="0.05"/>
 	<xacro:property name="cameraOffsetX" value="0.095"/>
+	<xacro:property name="cameraOffsetZ" value="0.06"/>
 </robot>

File: my_robot_description/urdf/sensors.xacro (robot description, xacro)
@@ -20,7 +20,7 @@
               rpy="0 0 0"/>
       <geometry>
-        <box size="${cameraSize}
-                   ${cameraSize}
-                   ${cameraSize}"/>
+        <box size="${cameraLength}
+                   ${cameraWidth}
+                   ${cameraHeight}"/>
       </geometry>
     </collision>
@@ -29,7 +29,7 @@
               rpy="0 0 0"/>
       <geometry>
-        <box size="${cameraSize}
-                   ${cameraSize}
-                   ${cameraSize}"/>
+        <box size="${cameraLength}
+                   ${cameraWidth}
+                   ${cameraHeight}"/>
       </geometry>
       <material name="green"/>
@@ -40,12 +40,12 @@
               rpy="0 0 0"/>
       <box_inertia m="${cameraMass}"
-                   x="${cameraSize}"
-                   y="${cameraSize}"
-                   z="${cameraSize}" />
+                   x="${cameraLength}"
+                   y="${cameraWidth}"
+                   z="${cameraHeight}" />
     </inertial>
   </link>
   <joint name="camera_joint" type="fixed">
     <axis xyz="0 1 0" />
-    <origin xyz="${cameraOffsetX} 0 ${2*wheelRadius}"
+    <origin xyz="${cameraOffsetX} 0 ${cameraOffsetZ}"
             rpy="0 0 0"/>
     <parent link="chassis"/>

Commit message: FIX GAZEBO SIM

File: my_robot_description/urdf/my_robot_properties.xacro (robot description, xacro)
@@ -18,14 +18,17 @@
 	<xacro:property name="wheelOffsetY" value="0.037"/>
 	<!-- Hokuyo laser properties -->
-	<xacro:property name="hokuyoMass" value="1e-5"/>
+	<xacro:property name="hokuyoMass" value="0.01"/>
 	<xacro:property name="hokuyoLength" value="0.05"/>
 	<xacro:property name="hokuyoWidth" value="0.05"/>
 	<xacro:property name="hokuyoHeight" value="0.07"/>
-	<xacro:property name="hokuyoOffsetZ" value="0.1125"/>
+	<xacro:property name="hokuyoOffsetX" value="0.035"/>
+	<!--xacro:property name="hokuyoOffsetX" value="0.05"/-->
+	<xacro:property name="hokuyoOffsetZ" value="0.1135"/>
+	<!--xacro:property name="hokuyoOffsetZ" value="0.1125"/-->
 	<!-- Camera properties -->
 	<xacro:property name="cameraLength" value="0.04"/>
 	<xacro:property name="cameraWidth" value="0.08"/>
 	<xacro:property name="cameraHeight" value="0.03"/>
-	<xacro:property name="cameraMass" value="0.05"/>
+	<xacro:property name="cameraMass" value="0.01"/>
 	<xacro:property name="cameraOffsetX" value="0.095"/>
 	<xacro:property name="cameraOffsetZ" value="0.06"/>

File: my_robot_description/urdf/sensors.xacro (robot description, xacro)
@@ -54,5 +54,5 @@
   <joint name="hokuyo_joint" type="fixed">
     <axis xyz="0 1 0" />
-    <origin xyz="0 0 ${hokuyoOffsetZ}"
+    <origin xyz="${hokuyoOffsetX} 0 ${hokuyoOffsetZ}"
             rpy="0 0 0"/>
     <parent link="chassis"/>
